File: ESP32-S2_Dev/ESP32-S2_Dev.sch (KiCad schematic (older format))
At the start: 114 parts, among them Q1 MMBT3906, Q2 BCW66GLT1G, Q3 BCW66GLT1G, U1 CP2102N-A01-GQFN28, U2 BD00C0AWFPS-ME2, U3 ESP32-S2, Y1 KC2520C40.0000C2YE00, Y2 Crystal

Commit message: fixed the oscillator footprint mirror issue, made Q1 a SOT416, and added power input diodes
Parts:
- added D4, D5: B120-E3, Diode_SMD:D_SMA, symbol Diode:B120-E3
- Q1: footprint Package_TO_SOT_SMD:SOT-23 -> Package_TO_SOT_SMD:SOT-416
- Y2: MOUSER (none) -> https://www.mouser.com/ProductDetail/?qs=byeeYqUIh0Mjq6I26A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
Connections:
- net USB_5P0: now also D4.1 (K), D5.1 (K); no longer C10.2, C11.2, C14.2, C16.2, D2.4 (K), D3.4 (K), UART1.1 (VBUS), USB1.1 (VBUS)
- new net: C11.2, C16.2, D3.4 (K), D5.2 (A), UART1.1 (VBUS)
- new net: C10.2, C14.2, D2.4 (K), D4.2 (A), USB1.1 (VBUS)
Other:
- note added: "Rev B Notes:\nAdd diode between usb inputs"
Changed lines of the file:
@@
 Title "ESP32-S2 DEV"
 Date "2022-04-28"
-Rev "00"
+Rev "01"
 Comp "Evil Geniuses for a better tommorrow"
 Comment1 ""
@@
 F 0 "Q1" H 1841 1154 50  0000 L CNN
 F 1 "MMBT3906" H 1300 1350 50  0000 L CNN
-F 2 "Package_TO_SOT_SMD:SOT-23" H 1850 1125 50  0001 L CIN
+F 2 "Package_TO_SOT_SMD:SOT-416" H 1850 1125 50  0001 L CIN
 F 3 "https://www.fairchildsemi.com/datasheets/2N/2N3906.pdf" H 1650 1200 50  0001 L CNN
 	1    1650 1200
@@
 Text Label 1100 2650 2    50   ~ 0
 USB_5P0
-Text Label 3150 3750 0    50   ~ 0
+Text Label 3550 3700 0    50   ~ 0
 USB_5P0
 Text Label 2250 3950 0    50   ~ 0
@@
 Text Label 2100 5800 2    50   ~ 0
 USB_DMinus
-Text Label 2100 6000 2    50   ~ 0
-USB_5P0
 $Comp
 L Device:C_Small C2
@@
 Wire Wire Line
 	2900 8400 2650 8400
-Text Label 3050 8200 0    50   ~ 0
+Text Label 3400 8100 0    50   ~ 0
 USB_5P0
 Text Label 2150 8400 0    50   ~ 0
@@
 LD0_3P3
 $Comp
-L bub_oscillators:KC2520C40.0000C2YE00 Y1
-U 1 1 62861CAB
-P 1700 9650
-F 0 "Y1" H 1700 9800 50  0000 C CNN
-F 1 "KC2520C40.0000C2YE00" H 1750 9250 50  0000 C CNN
-F 2 "bub_oscillators:KC2520C40.0000C2YE00" H 1850 8900 50  0001 C CNN
-F 3 "https://ele.kyocera.com/sites/default/files/assets/static/nrnd/kc2520c_c2_2019_e.pdf" H 1700 9650 50  0001 C CNN
-F 4 "https://www.digikey.com/en/products/detail/kyocera-avx/KC2520C40-0000C2YE00/2506201" H 1850 9050 50  0001 C CNN "Digikey"
-	1    1700 9650
-	1    0    0    -1
-$EndComp
-$Comp
 L Device:C_Small C9
 U 1 1 62862951
@@
 F 4 "https://www.digikey.com/en/products/detail/citizen-finedevice-co-ltd/CM315D-32-768KDZF-T/13663659" H 2000 10950 50  0001 C CNN "Digikey"
 F 5 "10095006" H 2000 10950 50  0001 C CNN "XESPN"
+F 6 "https://www.mouser.com/ProductDetail/?qs=byeeYqUIh0Mjq6I26A6tsQ%3D%3D" H 2000 10950 50  0001 C CNN "MOUSER"
 	1    2000 10950
 	-1   0    0    1
@@
 Wire Notes Line
 	8150 11450 8150 9250
+Text Notes 12100 8400 0    315  ~ 63
+Rev B Notes:\nAdd diode between usb inputs
+$Comp
+L bub_oscillators:KC2520C40.0000C2YE00 Y1
+U 1 1 62AAEBF0
+P 1700 9650
+F 0 "Y1" H 1700 9875 50  0000 C CNN
+F 1 "KC2520C40.0000C2YE00" H 1700 9784 50  0000 C CNN
+F 2 "bub_oscillators:KC2520C40.0000C2YE00" H 1850 8900 50  0001 C CNN
+F 3 "https://ele.kyocera.com/sites/default/files/assets/static/nrnd/kc2520c_c2_2019_e.pdf" H 1700 9650 50  0001 C CNN
+F 4 "https://www.digikey.com/en/products/detail/kyocera-avx/KC2520C40-0000C2YE00/2506201" H 1850 9050 50  0001 C CNN "Digikey"
+	1    1700 9650
+	1    0    0    -1
+$EndComp
+$Comp
+L Diode:B120-E3 D5
+U 1 1 62ACD5DC
+P 3400 3700
+F 0 "D5" H 3400 3483 50  0000 C CNN
+F 1 "B120-E3" H 3400 3574 50  0000 C CNN
+F 2 "Diode_SMD:D_SMA" H 3400 3525 50  0001 C CNN
+F 3 "http://www.vishay.com/docs/88946/b120.pdf" H 3400 3700 50  0001 C CNN
+	1    3400 3700
+	-1   0    0    1
+$EndComp
+Wire Wire Line
+	3250 3700 3150 3700
+Wire Wire Line
+	3150 3700 3150 3750
+Connection ~ 3150 3750
+$Comp
+L Diode:B120-E3 D4
+U 1 1 62AE48BA
+P 3250 8100
+F 0 "D4" H 3250 7883 50  0000 C CNN
+F 1 "B120-E3" H 3250 7974 50  0000 C CNN
+F 2 "Diode_SMD:D_SMA" H 3250 7925 50  0001 C CNN
+F 3 "http://www.vishay.com/docs/88946/b120.pdf" H 3250 8100 50  0001 C CNN
+	1    3250 8100
+	-1   0    0    1
+$EndComp
+Wire Wire Line
+	3100 8100 3100 8200
+Wire Wire Line
+	3100 8200 3050 8200
+Connection ~ 3050 8200
+Text Label 2100 6000 3    50   ~ 0
+USB_5P0
 $EndSCHEMATC

Commit message: fixed RTS and DTR and added them as well as the reset timing capacitors to the layout
Parts:
- added C37: 0.1u, Capacitor_SMD:C_0402_1005Metric, symbol Device:C_Small
- added R9: 10k, Resistor_SMD:R_0402_1005Metric, symbol Device:R_Small_US
Connections:
- net DTR: now also Q3.1 (E), R21.2; no longer Q2.1 (E), R22.2
- net GND: now also C37.2
- net MCU_3P3: now also R9.2
- net RST_PROG: now also C37.1, R9.1
- net RTS: now also Q2.1 (E), R22.2; no longer Q3.1 (E), R21.2
Other:
- note removed: "Rev B Notes:\nAdd diode between usb inputs"
- moved on the sheet: R37, RST1
Changed lines of the file:
@@
 Wire Wire Line
 	3700 3950 3850 3950
+Text Label 3700 3950 2    50   ~ 0
+DTR
 Text Label 3600 4700 2    50   ~ 0
-DTR
-Text Label 3700 3950 2    50   ~ 0
 RTS
 Wire Wire Line
@@
 	1    0    0    1
 $EndComp
-Text Label 5400 9650 0    50   ~ 0
+Text Label 7100 9950 0    50   ~ 0
 RST_PROG
 Text Label 6050 9650 0    50   ~ 0
@@
 L Device:R_Small_US R37
 U 1 1 629CE8DE
-P 5400 9750
-F 0 "R37" H 5600 9700 50  0000 R CNN
-F 1 "470" H 5600 9800 50  0000 R CNN
-F 2 "Resistor_SMD:R_0402_1005Metric" H 5400 9750 50  0001 C CNN
-F 3 "~" H 5400 9750 50  0001 C CNN
-	1    5400 9750
+P 7100 10150
+F 0 "R37" H 7300 10100 50  0000 R CNN
+F 1 "470" H 7300 10200 50  0000 R CNN
+F 2 "Resistor_SMD:R_0402_1005Metric" H 7100 10150 50  0001 C CNN
+F 3 "~" H 7100 10150 50  0001 C CNN
+	1    7100 10150
 	-1   0    0    1
 $EndComp
@@
 L Switch:SW_SPST RST1
 U 1 1 629DA67B
-P 5400 10050
-F 0 "RST1" V 5354 10148 50  0000 L CNN
-F 1 "B3U-1000P" V 5445 10148 50  0000 L CNN
-F 2 "Button_Switch_SMD:SW_SPST_B3U-1000P" H 5400 10050 50  0001 C CNN
-F 3 "https://omronfs.omron.com/en_US/ecb/products/pdf/en-b3u.pdf" H 5400 10050 50  0001 C CNN
-F 4 "https://www.digikey.com/en/products/detail/omron-electronics-inc-emc-div/B3U-1000P/1534338" V 5400 10050 50  0001 C CNN "DigiKey"
-	1    5400 10050
+P 7100 10450
+F 0 "RST1" V 7054 10548 50  0000 L CNN
+F 1 "B3U-1000P" V 7145 10548 50  0000 L CNN
+F 2 "Button_Switch_SMD:SW_SPST_B3U-1000P" H 7100 10450 50  0001 C CNN
+F 3 "https://omronfs.omron.com/en_US/ecb/products/pdf/en-b3u.pdf" H 7100 10450 50  0001 C CNN
+F 4 "https://www.digikey.com/en/products/detail/omron-electronics-inc-emc-div/B3U-1000P/1534338" V 7100 10450 50  0001 C CNN "DigiKey"
+	1    7100 10450
 	0    1    1    0
 $EndComp
@@
 L power:GND #PWR044
 U 1 1 629DB7E6
-P 5400 10250
-F 0 "#PWR044" H 5400 10000 50  0001 C CNN
-F 1 "GND" H 5405 10077 50  0000 C CNN
-F 2 "" H 5400 10250 50  0001 C CNN
-F 3 "" H 5400 10250 50  0001 C CNN
-	1    5400 10250
+P 7100 10650
+F 0 "#PWR044" H 7100 10400 50  0001 C CNN
+F 1 "GND" H 7105 10477 50  0000 C CNN
+F 2 "" H 7100 10650 50  0001 C CNN
+F 3 "" H 7100 10650 50  0001 C CNN
+	1    7100 10650
 	-1   0    0    -1
 $EndComp
@@
 Wire Notes Line
 	8150 11450 8150 9250
-Text Notes 12100 8400 0    315  ~ 63
-Rev B Notes:\nAdd diode between usb inputs
 $Comp
 L bub_oscillators:KC2520C40.0000C2YE00 Y1
@@
 Text Label 2100 6000 3    50   ~ 0
 USB_5P0
+$Comp
+L Device:R_Small_US R9
+U 1 1 62B4B318
+P 7100 9750
+F 0 "R9" H 7300 9700 50  0000 R CNN
+F 1 "10k" H 7300 9800 50  0000 R CNN
+F 2 "Resistor_SMD:R_0402_1005Metric" H 7100 9750 50  0001 C CNN
+F 3 "~" H 7100 9750 50  0001 C CNN
+	1    7100 9750
+	-1   0    0    1
+$EndComp
+Wire Wire Line
+	7100 9850 7100 10000
+Text Label 7100 9650 2    50   ~ 0
+MCU_3P3
+$Comp
+L Device:C_Small C37
+U 1 1 62B6247E
+P 7500 10100
+F 0 "C37" V 7400 10100 50  0000 R CNN
+F 1 "0.1u" V 7400 10300 50  0000 R CNN
+F 2 "Capacitor_SMD:C_0402_1005Metric" H 7500 10100 50  0001 C CNN
+F 3 "~" H 7500 10100 50  0001 C CNN
+	1    7500 10100
+	-1   0    0    -1
+$EndComp
+$Comp
+L power:GND #PWR0101
+U 1 1 62B62B2B
+P 7500 10200
+F 0 "#PWR0101" H 7500 9950 50  0001 C CNN
+F 1 "GND" H 7505 10027 50  0000 C CNN
+F 2 "" H 7500 10200 50  0001 C CNN
+F 3 "" H 7500 10200 50  0001 C CNN
+	1    7500 10200
+	-1   0    0    -1
+$EndComp
+Wire Wire Line
+	7500 10000 7100 10000
+Connection ~ 7100 10000
+Wire Wire Line
+	7100 10000 7100 10050
 $EndSCHEMATC

Commit message: changed flash to gigadevice, since microchip is not supported
Parts:
- removed SPI_FLASH_16Mb1: SST25VF016B-50-4I-QAF, Bub_flash:SST25VF016B-50-4I-QAF, symbol BubbaFlash:SST25VF016B-50-4I-QAF
- added U4: SPI_FLASH_8MEG, Bub_flash:USON8(2X3), symbol BubbaFlash:GD25WD80CEIGR
Connections:
- net GND: now also U4.4 (VSS)
- net MCU_3P3: now also U4.8 (VCC)
- net SPICLK: now also U4.6 (SCLK)
- net SPICS0: now also U4.1 (CS#)
- net SPID: now also U4.5 (SI)
- net SPIQ: now also U4.2 (SO)
- net SPIWP: now also U4.3 (WP#)
Changed lines of the file:
@@
 Text Label 1450 13900 2    50   ~ 0
 SPIWP
-Text Label 2650 13800 0    50   ~ 0
-SPIHD
 Text Label 1150 13700 2    50   ~ 0
 SPICS0
@@
 	-1   0    0    -1
 $EndComp
-Wire Wire Line
-	1450 14000 1350 14000
 Text Label 3500 13700 0    50   ~ 0
 MCU_3P3
@@
 	-1   0    0    -1
 $EndComp
-Wire Wire Line
-	2650 13700 3200 13700
 Connection ~ 3200 13700
 Wire Wire Line
 	3200 13700 3500 13700
-$Comp
-L BubbaFlash:SST25VF016B-50-4I-QAF SPI_FLASH_16Mb1
-U 1 1 6291918E
-P 1950 13600
-F 0 "SPI_FLASH_16Mb1" H 2000 13650 50  0000 C CNN
-F 1 "SST25VF016B-50-4I-QAF" H 2050 13100 50  0000 C CNN
-F 2 "Bub_flash:SST25VF016B-50-4I-QAF" H 1750 13600 50  0001 C CNN
-F 3 "https://ww1.microchip.com/downloads/en/DeviceDoc/20005044C.pdf" H 1750 13600 50  0001 C CNN
-F 4 "https://www.digikey.com/en/products/detail/microchip-technology/SST25VF016B-50-4I-QAF/2297795" H 1950 13600 50  0001 C CNN "Digikey"
-	1    1950 13600
-	1    0    0    -1
-$EndComp
 $Comp
 L Device:R_Small_US R3
@@
 	1    0    0    -1
 $EndComp
-Wire Wire Line
-	1450 13700 1250 13700
 Wire Wire Line
 	1250 13600 1250 13700
@@
 Wire Wire Line
 	7100 10000 7100 10050
+$Comp
+L BubbaFlash:GD25WD80CEIGR U4
+U 1 1 62B065AB
+P 2250 13600
+F 0 "U4" H 2050 13765 50  0000 C CNN
+F 1 "SPI_FLASH_8MEG" H 2050 13674 50  0000 C CNN
+F 2 "Bub_flash:USON8(2X3)" H 2250 13600 50  0001 C CNN
+F 3 "file:///C:/Users/bleblanc/Downloads/gd25wd80c_rev1.3_20190912.pdf" H 2250 13600 50  0001 C CNN
+F 4 "https://www.digikey.com/en/products/detail/gigadevice-semiconductor-hk-limited/GD25WD80CEIGR/9484742" H 2250 13600 50  0001 C CNN "DIGIKEY"
+	1    2250 13600
+	1    0    0    -1
+$EndComp
+Wire Wire Line
+	2500 13700 3200 13700
+Wire Wire Line
+	1350 14000 1600 14000
+Wire Wire Line
+	1600 13900 1450 13900
+Wire Wire Line
+	1250 13700 1600 13700
+Wire Wire Line
+	2650 13900 2500 13900
+Wire Wire Line
+	2650 14000 2500 14000
+Wire Wire Line
+	1450 13800 1600 13800
 $EndSCHEMATC
